File: _saved_placa_rf_wifi.sch (KiCad schematic (older format))
At the start: 9 parts

Commit message: Placa de prueba finalizada, la eleccion de las conexiones fueron para optimizar el ruteo
Changed lines of the file:
@@
 Wire Wire Line
 	3700 3250 3900 3250
-Text GLabel 4350 3850 1    50   BiDi ~ 0
+Text GLabel 4650 4350 3    50   BiDi ~ 0
 MOSI
 Text GLabel 4450 3850 1    50   BiDi ~ 0
 MISO
-Text GLabel 4550 4350 3    50   BiDi ~ 0
+Text GLabel 4350 3850 1    50   BiDi ~ 0
 SCK
+Text GLabel 4650 3850 1    50   BiDi ~ 0
+TX
 Text GLabel 4550 3850 1    50   BiDi ~ 0
-TX
-Text GLabel 4650 3850 1    50   BiDi ~ 0
 RX
 $Comp
@@
 	1    0    0    -1
 $EndComp
-Text GLabel 4650 4350 3    50   BiDi ~ 0
+Text GLabel 4750 4350 3    50   BiDi ~ 0
 IRQ
-Text GLabel 4750 4350 3    50   BiDi ~ 0
+Text GLabel 4550 4350 3    50   BiDi ~ 0
 CSN
 NoConn ~ 3700 3150

Commit message: Se trasladaron los pines de 2 a 10, inconvenientes con GND
Changed lines of the file:
@@
 Text GLabel 4650 4350 3    50   BiDi ~ 0
 MOSI
+Text GLabel 4550 3850 1    50   BiDi ~ 0
+MISO
 Text GLabel 4450 3850 1    50   BiDi ~ 0
-MISO
-Text GLabel 4350 3850 1    50   BiDi ~ 0
 SCK
+Text GLabel 4750 3850 1    50   BiDi ~ 0
+TX
 Text GLabel 4650 3850 1    50   BiDi ~ 0
-TX
-Text GLabel 4550 3850 1    50   BiDi ~ 0
 RX
 $Comp
@@
 CSN
 NoConn ~ 3700 3150
-NoConn ~ 4750 3850
+NoConn ~ 4350 3850
 $EndSCHEMATC
