File: placa_rf_wifi.sch (KiCad schematic (older format))
At the start: 9 parts

Commit message: Version de la placa simplificada, con un solo LED
Changed lines of the file:
@@
 Text GLabel 4650 4350 3    50   BiDi ~ 0
 MOSI
+Text GLabel 4750 3850 1    50   BiDi ~ 0
+MISO
+Text GLabel 4650 3850 1    50   BiDi ~ 0
+SCK
+Text GLabel 4450 3850 1    50   BiDi ~ 0
+TX
 Text GLabel 4550 3850 1    50   BiDi ~ 0
-MISO
-Text GLabel 4450 3850 1    50   BiDi ~ 0
-SCK
-Text GLabel 4750 3850 1    50   BiDi ~ 0
-TX
-Text GLabel 4650 3850 1    50   BiDi ~ 0
 RX
 $Comp

Commit message: Placa simplificada II, nueva disposicion de pines
Connections:
- net labels added: CE
- no-connect marks 5 -> 3
Changed lines of the file:
@@
 Text GLabel 4650 3850 1    50   BiDi ~ 0
 SCK
+Text GLabel 4350 3850 1    50   BiDi ~ 0
+TX
 Text GLabel 4450 3850 1    50   BiDi ~ 0
-TX
-Text GLabel 4550 3850 1    50   BiDi ~ 0
 RX
 $Comp
@@
 Text GLabel 4550 4350 3    50   BiDi ~ 0
 CSN
-NoConn ~ 3700 3150
-NoConn ~ 4350 3850
+Text GLabel 3700 3150 2    50   BiDi ~ 0
+CE
+Text GLabel 4550 3850 1    50   BiDi ~ 0
+CE
 $EndSCHEMATC

Commit message: Placa simplificada II, sin IRQ y sin uso del RB8
Connections:
- net labels removed: IRQ
- no-connect marks 3 -> 5
Changed lines of the file:
@@
 Text GLabel 3700 2950 2    50   BiDi ~ 0
 MISO
-Text GLabel 3200 2950 0    50   BiDi ~ 0
-IRQ
 Wire Wire Line
 	2900 3250 3200 3250
@@
 Text GLabel 4650 4350 3    50   BiDi ~ 0
 MOSI
+Text GLabel 4750 4350 3    50   BiDi ~ 0
+MISO
 Text GLabel 4750 3850 1    50   BiDi ~ 0
-MISO
-Text GLabel 4650 3850 1    50   BiDi ~ 0
 SCK
-Text GLabel 4350 3850 1    50   BiDi ~ 0
+Text GLabel 4450 3850 1    50   BiDi ~ 0
 TX
-Text GLabel 4450 3850 1    50   BiDi ~ 0
+Text GLabel 4550 3850 1    50   BiDi ~ 0
 RX
 $Comp
@@
 	1    0    0    -1
 $EndComp
-Text GLabel 4750 4350 3    50   BiDi ~ 0
-IRQ
 Text GLabel 4550 4350 3    50   BiDi ~ 0
 CSN
 Text GLabel 3700 3150 2    50   BiDi ~ 0
 CE
-Text GLabel 4550 3850 1    50   BiDi ~ 0
+Text GLabel 4650 3850 1    50   BiDi ~ 0
 CE
+NoConn ~ 3200 2950
+NoConn ~ 4350 3850
 $EndSCHEMATC
